Commit message: Adapt urdf and xacro files so parent and origin can be forwarded.

File: flexiv_description/urdf/rizon.urdf.xacro (robot description, xacro)
@@ -22,4 +22,5 @@
     fake_sensor_commands="$(arg fake_sensor_commands)"
     initial_positions="${xacro.load_yaml(initial_positions_file)}">
+    <origin xyz="0.0 0.0 0.0" rpy="0 0 0"/>
   </xacro:rizon_robot>
 </robot>

File: flexiv_description/urdf/rizon10_joints_links.xacro (robot description, xacro)
@@ -7,10 +7,15 @@
     NOTE: accurate kinematic but approximated dynamics parameters
   -->
-  <xacro:macro name="rizon10_joints_links" params="rizon_type prefix mesh_prefix_path">
+  <xacro:macro name="rizon10_joints_links" params="rizon_type prefix mesh_prefix_path add_world:=true parent:=world *origin ">
     <!-- JOINTS-->
     <joint name="${prefix}base_joint" type="fixed">
-      <parent link="world"/>
+      <xacro:if value="${add_world}">
+        <parent link="world"/>
+      </xacro:if>
+      <xacro:unless value="${add_world}">
+        <parent link="${parent}"/>
+      </xacro:unless>
       <child link="${prefix}base_link" />
-      <origin xyz="0.0 0.0 0.0" rpy="0.0 0.0 0.0"/>
+      <xacro:insert_block name="origin" />
     </joint>
     <joint name="${prefix}joint1" type="revolute">
@@ -74,6 +79,8 @@
     </joint>
     <!-- LINKS -->
-    <link name="world">
-    </link>
+    <xacro:if value="${add_world}">
+      <link name="world">
+      </link>
+    </xacro:if>
     <link name="${prefix}base_link">
       <inertial>

File: flexiv_description/urdf/rizon4_joints_links.xacro (robot description, xacro)
@@ -7,10 +7,15 @@
     NOTE: accurate kinematic but approximated dynamics parameters
   -->
-  <xacro:macro name="rizon4_joints_links" params="rizon_type prefix mesh_prefix_path">
+  <xacro:macro name="rizon4_joints_links" params="rizon_type prefix mesh_prefix_path add_world:=true parent:=world *origin ">
     <!-- JOINTS-->
     <joint name="${prefix}base_joint" type="fixed">
-      <parent link="world"/>
+      <xacro:if value="${add_world}">
+        <parent link="world"/>
+      </xacro:if>
+      <xacro:unless value="${add_world}">
+        <parent link="${parent}"/>
+      </xacro:unless>
       <child link="${prefix}base_link" />
-      <origin xyz="0.0 0.0 0.0" rpy="0.0 0.0 0.0"/>
+      <xacro:insert_block name="origin" />
     </joint>
     <joint name="${prefix}joint1" type="revolute">
@@ -74,6 +79,8 @@
     </joint>
     <!-- LINKS -->
-    <link name="world">
-    </link>
+    <xacro:if value="${add_world}">
+      <link name="world">
+      </link>
+    </xacro:if>
     <link name="${prefix}base_link">
       <inertial>

File: flexiv_description/urdf/rizon_macro.xacro (robot description, xacro)
@@ -5,7 +5,10 @@
     prefix
     robot_sn
+    *origin
     use_fake_hardware:=false
     fake_sensor_commands:=false
     initial_positions:=${dict(joint1=0.0,joint2=-0.69813,joint3=0.0,joint4=1.570796,joint5=0.0,joint6=0.69813,joint7=0.0)}
+    add_world:=true
+    parent:=world
     ">
     <!-- Import Rviz colors -->
@@ -14,5 +17,8 @@
     <xacro:if value="${rizon_type=='rizon4' or rizon_type=='rizon4s'}">
       <xacro:include filename="$(find flexiv_description)/urdf/rizon4_joints_links.xacro" />
-      <xacro:rizon4_joints_links rizon_type="${rizon_type}" prefix="${prefix}" mesh_prefix_path="package://flexiv_description/" />
+      <xacro:rizon4_joints_links rizon_type="${rizon_type}" prefix="${prefix}" mesh_prefix_path="package://flexiv_description/"
+                                 add_world="${add_world}" parent="${parent}">
+        <xacro:insert_block name="origin" />
+      </xacro:rizon4_joints_links>
       <!-- ros2 control include -->
       <xacro:include filename="$(find flexiv_description)/urdf/rizon4.ros2_control.xacro"/>
@@ -26,5 +32,8 @@
     <xacro:if value="${rizon_type=='rizon10' or rizon_type=='rizon10s'}">
       <xacro:include filename="$(find flexiv_description)/urdf/rizon10_joints_links.xacro" />
-      <xacro:rizon10_joints_links rizon_type="${rizon_type}" prefix="${prefix}" mesh_prefix_path="package://flexiv_description/" />
+      <xacro:rizon10_joints_links rizon_type="${rizon_type}" prefix="${prefix}" mesh_prefix_path="package://flexiv_description/"
+                                  add_world="${add_world}" parent="${parent}">
+        <xacro:insert_block name="origin" />
+      </xacro:rizon10_joints_links>
       <!-- ros2 control include -->
       <xacro:include filename="$(find flexiv_description)/urdf/rizon10.ros2_control.xacro"/>

Commit message: Adapt urdf and xacro files so parent and origin can be forwarded.

File: flexiv_description/urdf/rizon.urdf.xacro (robot description, xacro)
@@ -24,4 +24,5 @@
     fake_sensor_commands="$(arg fake_sensor_commands)"
     initial_positions="${xacro.load_yaml(initial_positions_file)}">
+    <origin xyz="0.0 0.0 0.0" rpy="0 0 0"/>
   </xacro:rizon_robot>
 </robot>

File: flexiv_description/urdf/rizon10_joints_links.xacro (robot description, xacro)
@@ -7,10 +7,15 @@
     NOTE: accurate kinematic but approximated dynamics parameters
   -->
-  <xacro:macro name="rizon10_joints_links" params="rizon_type prefix mesh_prefix_path">
+  <xacro:macro name="rizon10_joints_links" params="rizon_type prefix mesh_prefix_path add_world:=true parent:=world *origin ">
     <!-- JOINTS-->
     <joint name="${prefix}base_joint" type="fixed">
-      <parent link="world"/>
+      <xacro:if value="${add_world}">
+        <parent link="world"/>
+      </xacro:if>
+      <xacro:unless value="${add_world}">
+        <parent link="${parent}"/>
+      </xacro:unless>
       <child link="${prefix}base_link" />
-      <origin xyz="0.0 0.0 0.0" rpy="0.0 0.0 0.0"/>
+      <xacro:insert_block name="origin" />
     </joint>
     <joint name="${prefix}joint1" type="revolute">
@@ -69,6 +74,8 @@
     </joint>
     <!-- LINKS -->
-    <link name="world">
-    </link>
+    <xacro:if value="${add_world}">
+      <link name="world">
+      </link>
+    </xacro:if>
     <link name="${prefix}base_link">
       <inertial>

File: flexiv_description/urdf/rizon4_joints_links.xacro (robot description, xacro)
@@ -7,10 +7,15 @@
     NOTE: accurate kinematic but approximated dynamics parameters
   -->
-  <xacro:macro name="rizon4_joints_links" params="rizon_type prefix mesh_prefix_path">
+  <xacro:macro name="rizon4_joints_links" params="rizon_type prefix mesh_prefix_path add_world:=true parent:=world *origin ">
     <!-- JOINTS-->
     <joint name="${prefix}base_joint" type="fixed">
-      <parent link="world"/>
+      <xacro:if value="${add_world}">
+        <parent link="world"/>
+      </xacro:if>
+      <xacro:unless value="${add_world}">
+        <parent link="${parent}"/>
+      </xacro:unless>
       <child link="${prefix}base_link" />
-      <origin xyz="0.0 0.0 0.0" rpy="0.0 0.0 0.0"/>
+      <xacro:insert_block name="origin" />
     </joint>
     <joint name="${prefix}joint1" type="revolute">
@@ -74,6 +79,8 @@
     </joint>
     <!-- LINKS -->
-    <link name="world">
-    </link>
+    <xacro:if value="${add_world}">
+      <link name="world">
+      </link>
+    </xacro:if>
     <link name="${prefix}base_link">
       <inertial>

File: flexiv_description/urdf/rizon_macro.xacro (robot description, xacro)
@@ -8,5 +8,8 @@
     use_fake_hardware:=false
     fake_sensor_commands:=false
+    *origin
     initial_positions:=${dict(joint1=0.0,joint2=-0.69813,joint3=0.0,joint4=1.570796,joint5=0.0,joint6=0.69813,joint7=0.0)}
+    add_world:=true
+    parent:=world
     ">
     <!-- Import Rviz colors -->
@@ -15,5 +18,8 @@
     <xacro:if value="${rizon_type=='rizon4' or rizon_type=='rizon4s'}">
       <xacro:include filename="$(find flexiv_description)/urdf/rizon4_joints_links.xacro" />
-      <xacro:rizon4_joints_links rizon_type="${rizon_type}" prefix="${prefix}" mesh_prefix_path="package://flexiv_description/" />
+      <xacro:rizon4_joints_links rizon_type="${rizon_type}" prefix="${prefix}" mesh_prefix_path="package://flexiv_description/"
+                                 add_world="${add_world}" parent="${parent}">
+        <xacro:insert_block name="origin" />
+      </xacro:rizon4_joints_links>
       <!-- ros2 control include -->
       <xacro:include filename="$(find flexiv_description)/urdf/rizon4.ros2_control.xacro"/>
@@ -27,5 +33,8 @@
     <xacro:if value="${rizon_type=='rizon10'}">
       <xacro:include filename="$(find flexiv_description)/urdf/rizon10_joints_links.xacro" />
-      <xacro:rizon10_joints_links rizon_type="${rizon_type}" prefix="${prefix}" mesh_prefix_path="package://flexiv_description/" />
+      <xacro:rizon10_joints_links rizon_type="${rizon_type}" prefix="${prefix}" mesh_prefix_path="package://flexiv_description/"
+                                  add_world="${add_world}" parent="${parent}">
+        <xacro:insert_block name="origin" />
+      </xacro:rizon10_joints_links>
       <!-- ros2 control include -->
       <xacro:include filename="$(find flexiv_description)/urdf/rizon10.ros2_control.xacro"/>

Commit message: Adapt urdf and xacro files so parent and origin can be forwarded.

File: flexiv_description/urdf/rizon.urdf.xacro (robot description, xacro)
@@ -24,4 +24,5 @@
     fake_sensor_commands="$(arg fake_sensor_commands)"
     initial_positions="${xacro.load_yaml(initial_positions_file)}">
+    <origin xyz="0.0 0.0 0.0" rpy="0 0 0"/>
   </xacro:rizon_robot>
 </robot>

File: flexiv_description/urdf/rizon_macro.xacro (robot description, xacro)
@@ -8,5 +8,8 @@
     use_fake_hardware:=false
     fake_sensor_commands:=false
+    *origin
     initial_positions:=${dict(joint1=0.0,joint2=-0.69813,joint3=0.0,joint4=1.570796,joint5=0.0,joint6=0.69813,joint7=0.0)}
+    add_world:=true
+    parent:=world
     ">
     <!-- Load gripper -->
@@ -20,5 +23,8 @@
     <xacro:if value="${rizon_type=='rizon4' or rizon_type=='rizon4s'}">
       <xacro:include filename="$(find flexiv_description)/urdf/rizon4_joints_links.xacro" />
-      <xacro:rizon4_joints_links rizon_type="${rizon_type}" prefix="${prefix}" mesh_prefix_path="package://flexiv_description/" />
+      <xacro:rizon4_joints_links rizon_type="${rizon_type}" prefix="${prefix}" mesh_prefix_path="package://flexiv_description/"
+                                 add_world="${add_world}" parent="${parent}">
+        <xacro:insert_block name="origin" />
+      </xacro:rizon4_joints_links>
       <!-- ros2 control include -->
       <xacro:include filename="$(find flexiv_description)/urdf/rizon4.ros2_control.xacro"/>
@@ -32,5 +38,8 @@
     <xacro:if value="${rizon_type=='rizon10' or rizon_type=='rizon10s'}">
       <xacro:include filename="$(find flexiv_description)/urdf/rizon10_joints_links.xacro" />
-      <xacro:rizon10_joints_links rizon_type="${rizon_type}" prefix="${prefix}" mesh_prefix_path="package://flexiv_description/" />
+      <xacro:rizon10_joints_links rizon_type="${rizon_type}" prefix="${prefix}" mesh_prefix_path="package://flexiv_description/"
+                                  add_world="${add_world}" parent="${parent}">
+        <xacro:insert_block name="origin" />
+      </xacro:rizon10_joints_links>
       <!-- ros2 control include -->
       <xacro:include filename="$(find flexiv_description)/urdf/rizon10.ros2_control.xacro"/>
