Commit message: mujoco: give link collisions unique names

File: flexiv_description/urdf/rizon4_joints_links.xacro (robot description, xacro)
@@ -96,5 +96,5 @@
         <material name="rizon_light_grey" />
       </visual>
-      <collision>
+      <collision name="${prefix}base_link">
         <origin xyz="0 0 0" rpy="0 0 0"/>
         <geometry>
@@ -116,5 +116,5 @@
         <material name="rizon_light_grey" />
       </visual>
-      <collision>
+      <collision name="${prefix}link1">
         <origin xyz="0 0 0" rpy="0 0 0" />
         <geometry>
@@ -136,5 +136,5 @@
         <material name="rizon_light_grey" />
       </visual>
-      <collision>
+      <collision name="${prefix}link2">
         <origin xyz="0 0 0" rpy="0 0 0"/>
         <geometry>
@@ -156,5 +156,5 @@
         <material name="rizon_light_grey" />
       </visual>
-      <collision>
+      <collision name="${prefix}link3">
         <origin xyz="0 0 0" rpy="0 0 0" />
         <geometry>
@@ -176,5 +176,5 @@
         <material name="rizon_light_grey" />
       </visual>
-      <collision>
+      <collision name="${prefix}link4">
         <origin xyz="0 0 0" rpy="0 0 0"/>
         <geometry>
@@ -196,5 +196,5 @@
         <material name="rizon_light_grey" />
       </visual>
-      <collision>
+      <collision name="${prefix}link5">
         <origin xyz="0 0 0" rpy="0 0 0"/>
         <geometry>
@@ -216,5 +216,5 @@
         <material name="rizon_light_grey" />
       </visual>
-      <collision>
+      <collision name="${prefix}link6">
         <origin xyz="0 0 0" rpy="0 0 0"/>
         <geometry>
@@ -237,5 +237,5 @@
           <material name="rizon_light_grey" />
         </visual>
-        <collision>
+        <collision name="${prefix}link7">
           <origin xyz="0 0 0" rpy="0 0 0"/>
           <geometry>
@@ -257,5 +257,5 @@
           <material name="rizon_light_grey" />
         </visual>
-        <collision>
+        <collision name="${prefix}link7">
           <origin xyz="0 0 0" rpy="0 0 0"/>
           <geometry>

Commit message: mujoco: give link collisions unique names

File: flexiv_description/urdf/rizon4_joints_links.xacro (robot description, xacro)
@@ -96,5 +96,5 @@
         <material name="rizon_light_grey" />
       </visual>
-      <collision name="hull">
+      <collision name="${prefix}base_link">
         <origin xyz="0 0 0" rpy="0 0 0"/>
         <geometry>
@@ -123,5 +123,5 @@
         <material name="rizon_white" />
       </visual>
-      <collision name="hull">
+      <collision name="${prefix}link1">
         <origin xyz="0 0 0" rpy="0 0 0" />
         <geometry>
@@ -150,5 +150,5 @@
         <material name="rizon_white" />
       </visual>
-      <collision name="hull">
+      <collision name="${prefix}link2">
         <origin xyz="0 0 0" rpy="0 0 0"/>
         <geometry>
@@ -177,5 +177,5 @@
         <material name="rizon_white" />
       </visual>
-      <collision name="hull">
+      <collision name="${prefix}link3">
         <origin xyz="0 0 0" rpy="0 0 0" />
         <geometry>
@@ -204,5 +204,5 @@
         <material name="rizon_white" />
       </visual>
-      <collision name="hull">
+      <collision name="${prefix}link4">
         <origin xyz="0 0 0" rpy="0 0 0"/>
         <geometry>
@@ -231,5 +231,5 @@
         <material name="rizon_white" />
       </visual>
-      <collision name="hull">
+      <collision name="${prefix}link5">
         <origin xyz="0 0 0" rpy="0 0 0"/>
         <geometry>
@@ -258,5 +258,5 @@
         <material name="rizon_white" />
       </visual>
-      <collision name="hull">
+      <collision name="${prefix}link6">
         <origin xyz="0 0 0" rpy="0 0 0"/>
         <geometry>
@@ -286,5 +286,5 @@
           <material name="rizon_white" />
         </visual>
-        <collision name="hull">
+        <collision name="${prefix}link7">
           <origin xyz="0 0 0" rpy="0 0 0"/>
           <geometry>
@@ -313,5 +313,5 @@
           <material name="rizon_white" />
         </visual>
-        <collision name="hull">
+        <collision name="${prefix}link7">
           <origin xyz="0 0 0" rpy="0 0 0"/>
           <geometry>
