Commit message: introduce a ros2_control joint macro

File: flexiv_description/urdf/rizon4.ros2_control.xacro (robot description, xacro)
@@ -21,123 +21,33 @@
         </xacro:unless>
       </hardware>
-      <joint name="${prefix}joint1">
-        <command_interface name="position">
-          <param name="min">-2.7925</param>
-          <param name="max">2.7925</param>
-        </command_interface>
-        <command_interface name="velocity">
-          <param name="min">-2.0944</param>
-          <param name="max">2.0944</param>
-        </command_interface>
-        <command_interface name="effort"/>
-        <state_interface name="position">
-          <!-- initial position for the FakeSystem -->
-          <param name="initial_value">${initial_positions['joint1']}</param>
-        </state_interface>
-        <state_interface name="velocity"/>
-        <state_interface name="effort"/>
-      </joint>
-      <joint name="${prefix}joint2">
-        <command_interface name="position">
-          <param name="min">-2.2689</param>
-          <param name="max">2.2689</param>
-        </command_interface>
-        <command_interface name="velocity">
-          <param name="min">-2.0944</param>
-          <param name="max">2.0944</param>
-        </command_interface>
-        <command_interface name="effort"/>
-        <state_interface name="position">
-          <!-- initial position for the FakeSystem -->
-          <param name="initial_value">${initial_positions['joint2']}</param>
-        </state_interface>
-        <state_interface name="velocity"/>
-        <state_interface name="effort"/>
-      </joint>
-      <joint name="${prefix}joint3">
-        <command_interface name="position">
-          <param name="min">-2.9671</param>
-          <param name="max">2.9671</param>
-        </command_interface>
-        <command_interface name="velocity">
-          <param name="min">-2.4435</param>
-          <param name="max">2.4435</param>
-        </command_interface>
-        <command_interface name="effort"/>
-        <state_interface name="position">
-          <!-- initial position for the FakeSystem -->
-          <param name="initial_value">${initial_positions['joint3']}</param>
-        </state_interface>
-        <state_interface name="velocity"/>
-        <state_interface name="effort"/>
-      </joint>
-      <joint name="${prefix}joint4">
-        <command_interface name="position">
-          <param name="min">-1.8675</param>
-          <param name="max">2.6878</param>
-        </command_interface>
-        <command_interface name="velocity">
-          <param name="min">-2.4435</param>
-          <param name="max">2.4435</param>
-        </command_interface>
-        <command_interface name="effort"/>
-        <state_interface name="position">
-          <!-- initial position for the FakeSystem -->
-          <param name="initial_value">${initial_positions['joint4']}</param>
-        </state_interface>
-        <state_interface name="velocity"/>
-        <state_interface name="effort"/>
-      </joint>
-      <joint name="${prefix}joint5">
-        <command_interface name="position">
-          <param name="min">-2.9671</param>
-          <param name="max">2.9671</param>
-        </command_interface>
-        <command_interface name="velocity">
-          <param name="min">-4.8869</param>
-          <param name="max">4.8869</param>
-        </command_interface>
-        <command_interface name="effort"/>
-        <state_interface name="position">
-          <!-- initial position for the FakeSystem -->
-          <param name="initial_value">${initial_positions['joint5']}</param>
-        </state_interface>
-        <state_interface name="velocity"/>
-        <state_interface name="effort"/>
-      </joint>
-      <joint name="${prefix}joint6">
-        <command_interface name="position">
-          <param name="min">-1.3963</param>
-          <param name="max">4.5379</param>
-        </command_interface>
-        <command_interface name="velocity">
-          <param name="min">-4.8869</param>
-          <param name="max">4.8869</param>
-        </command_interface>
-        <command_interface name="effort"/>
-        <state_interface name="position">
-          <!-- initial position for the FakeSystem -->
-          <param name="initial_value">${initial_positions['joint6']}</param>
-        </state_interface>
-        <state_interface name="velocity"/>
-        <state_interface name="effort"/>
-      </joint>
-      <joint name="${prefix}joint7">
-        <command_interface name="position">
-          <param name="min">-2.9671</param>
-          <param name="max">2.9671</param>
-        </command_interface>
-        <command_interface name="velocity">
-          <param name="min">-4.8869</param>
-          <param name="max">4.8869</param>
-        </command_interface>
-        <command_interface name="effort"/>
-        <state_interface name="position">
-          <!-- initial position for the FakeSystem -->
-          <param name="initial_value">${initial_positions['joint7']}</param>
-        </state_interface>
-        <state_interface name="velocity"/>
-        <state_interface name="effort"/>
-      </joint>
+      <xacro:include filename="$(find flexiv_description)/urdf/joint.ros2_control.xacro"/>
+      <xacro:joint_ros2_control name="joint1"
+        initial_position="${initial_positions['joint1']}"
+        pos_min="-2.7925" pos_max="2.7925"
+        vel_min="-2.0944" vel_max="2.0944"/>
+      <xacro:joint_ros2_control name="joint2"
+        initial_position="${initial_positions['joint2']}"
+        pos_min="-2.2689" pos_max="2.2689"
+        vel_min="-2.0944" vel_max="2.0944"/>
+      <xacro:joint_ros2_control name="joint3"
+        initial_position="${initial_positions['joint3']}"
+        pos_min="-2.9671" pos_max="2.9671"
+        vel_min="-2.4435" vel_max="2.4435"/>
+      <xacro:joint_ros2_control name="joint4"
+        initial_position="${initial_positions['joint4']}"
+        pos_min="-1.8675" pos_max="2.6878"
+        vel_min="-2.4435" vel_max="2.4435"/>
+      <xacro:joint_ros2_control name="joint5"
+        initial_position="${initial_positions['joint5']}"
+        pos_min="-2.9671" pos_max="2.9671"
+        vel_min="-4.8869" vel_max="4.8869"/>
+      <xacro:joint_ros2_control name="joint6"
+        initial_position="${initial_positions['joint6']}"
+        pos_min="-1.3963" pos_max="4.5379"
+        vel_min="-4.8869" vel_max="4.8869"/>
+      <xacro:joint_ros2_control name="joint7"
+        initial_position="${initial_positions['joint7']}"
+        pos_min="-2.9671" pos_max="2.9671"
+        vel_min="-4.8869" vel_max="4.8869"/>
       <!-- 18 digital IO ports (16 on control box + 2 inside the wrist connector) -->
       <gpio name="${prefix}gpio">

Commit message: introduce a ros2_control joint macro

File: flexiv_description/urdf/rizon4.ros2_control.xacro (robot description, xacro)
@@ -23,123 +23,33 @@
         </xacro:unless>
       </hardware>
-      <joint name="${prefix}joint1">
-        <command_interface name="position">
-          <param name="min">-2.7925</param>
-          <param name="max">2.7925</param>
-        </command_interface>
-        <command_interface name="velocity">
-          <param name="min">-2.0944</param>
-          <param name="max">2.0944</param>
-        </command_interface>
-        <command_interface name="effort"/>
-        <state_interface name="position">
-          <!-- initial position for the FakeSystem -->
-          <param name="initial_value">${initial_positions['joint1']}</param>
-        </state_interface>
-        <state_interface name="velocity"/>
-        <state_interface name="effort"/>
-      </joint>
-      <joint name="${prefix}joint2">
-        <command_interface name="position">
-          <param name="min">-2.2689</param>
-          <param name="max">2.2689</param>
-        </command_interface>
-        <command_interface name="velocity">
-          <param name="min">-2.0944</param>
-          <param name="max">2.0944</param>
-        </command_interface>
-        <command_interface name="effort"/>
-        <state_interface name="position">
-          <!-- initial position for the FakeSystem -->
-          <param name="initial_value">${initial_positions['joint2']}</param>
-        </state_interface>
-        <state_interface name="velocity"/>
-        <state_interface name="effort"/>
-      </joint>
-      <joint name="${prefix}joint3">
-        <command_interface name="position">
-          <param name="min">-2.9671</param>
-          <param name="max">2.9671</param>
-        </command_interface>
-        <command_interface name="velocity">
-          <param name="min">-2.4435</param>
-          <param name="max">2.4435</param>
-        </command_interface>
-        <command_interface name="effort"/>
-        <state_interface name="position">
-          <!-- initial position for the FakeSystem -->
-          <param name="initial_value">${initial_positions['joint3']}</param>
-        </state_interface>
-        <state_interface name="velocity"/>
-        <state_interface name="effort"/>
-      </joint>
-      <joint name="${prefix}joint4">
-        <command_interface name="position">
-          <param name="min">-1.8675</param>
-          <param name="max">2.6878</param>
-        </command_interface>
-        <command_interface name="velocity">
-          <param name="min">-2.4435</param>
-          <param name="max">2.4435</param>
-        </command_interface>
-        <command_interface name="effort"/>
-        <state_interface name="position">
-          <!-- initial position for the FakeSystem -->
-          <param name="initial_value">${initial_positions['joint4']}</param>
-        </state_interface>
-        <state_interface name="velocity"/>
-        <state_interface name="effort"/>
-      </joint>
-      <joint name="${prefix}joint5">
-        <command_interface name="position">
-          <param name="min">-2.9671</param>
-          <param name="max">2.9671</param>
-        </command_interface>
-        <command_interface name="velocity">
-          <param name="min">-4.8869</param>
-          <param name="max">4.8869</param>
-        </command_interface>
-        <command_interface name="effort"/>
-        <state_interface name="position">
-          <!-- initial position for the FakeSystem -->
-          <param name="initial_value">${initial_positions['joint5']}</param>
-        </state_interface>
-        <state_interface name="velocity"/>
-        <state_interface name="effort"/>
-      </joint>
-      <joint name="${prefix}joint6">
-        <command_interface name="position">
-          <param name="min">-1.3963</param>
-          <param name="max">4.5379</param>
-        </command_interface>
-        <command_interface name="velocity">
-          <param name="min">-4.8869</param>
-          <param name="max">4.8869</param>
-        </command_interface>
-        <command_interface name="effort"/>
-        <state_interface name="position">
-          <!-- initial position for the FakeSystem -->
-          <param name="initial_value">${initial_positions['joint6']}</param>
-        </state_interface>
-        <state_interface name="velocity"/>
-        <state_interface name="effort"/>
-      </joint>
-      <joint name="${prefix}joint7">
-        <command_interface name="position">
-          <param name="min">-2.9671</param>
-          <param name="max">2.9671</param>
-        </command_interface>
-        <command_interface name="velocity">
-          <param name="min">-4.8869</param>
-          <param name="max">4.8869</param>
-        </command_interface>
-        <command_interface name="effort"/>
-        <state_interface name="position">
-          <!-- initial position for the FakeSystem -->
-          <param name="initial_value">${initial_positions['joint7']}</param>
-        </state_interface>
-        <state_interface name="velocity"/>
-        <state_interface name="effort"/>
-      </joint>
+      <xacro:include filename="$(find flexiv_description)/urdf/joint.ros2_control.xacro"/>
+      <xacro:joint_ros2_control name="joint1"
+        initial_position="${initial_positions['joint1']}"
+        pos_min="-2.7925" pos_max="2.7925"
+        vel_min="-2.0944" vel_max="2.0944"/>
+      <xacro:joint_ros2_control name="joint2"
+        initial_position="${initial_positions['joint2']}"
+        pos_min="-2.2689" pos_max="2.2689"
+        vel_min="-2.0944" vel_max="2.0944"/>
+      <xacro:joint_ros2_control name="joint3"
+        initial_position="${initial_positions['joint3']}"
+        pos_min="-2.9671" pos_max="2.9671"
+        vel_min="-2.4435" vel_max="2.4435"/>
+      <xacro:joint_ros2_control name="joint4"
+        initial_position="${initial_positions['joint4']}"
+        pos_min="-1.8675" pos_max="2.6878"
+        vel_min="-2.4435" vel_max="2.4435"/>
+      <xacro:joint_ros2_control name="joint5"
+        initial_position="${initial_positions['joint5']}"
+        pos_min="-2.9671" pos_max="2.9671"
+        vel_min="-4.8869" vel_max="4.8869"/>
+      <xacro:joint_ros2_control name="joint6"
+        initial_position="${initial_positions['joint6']}"
+        pos_min="-1.3963" pos_max="4.5379"
+        vel_min="-4.8869" vel_max="4.8869"/>
+      <xacro:joint_ros2_control name="joint7"
+        initial_position="${initial_positions['joint7']}"
+        pos_min="-2.9671" pos_max="2.9671"
+        vel_min="-4.8869" vel_max="4.8869"/>
       <sensor name="${prefix}force_torque_sensor">
         <state_interface name="force.x"/>

Commit message: add mujoco ros2_control

File: flexiv_description/urdf/rizon4.ros2_control.xacro (robot description, xacro)
@@ -21,33 +21,123 @@
         </xacro:unless>
       </hardware>
-      <xacro:include filename="$(find flexiv_description)/urdf/joint.ros2_control.xacro"/>
-      <xacro:joint_ros2_control name="joint1"
-        initial_position="${initial_positions['joint1']}"
-        pos_min="-2.7925" pos_max="2.7925"
-        vel_min="-2.0944" vel_max="2.0944"/>
-      <xacro:joint_ros2_control name="joint2"
-        initial_position="${initial_positions['joint2']}"
-        pos_min="-2.2689" pos_max="2.2689"
-        vel_min="-2.0944" vel_max="2.0944"/>
-      <xacro:joint_ros2_control name="joint3"
-        initial_position="${initial_positions['joint3']}"
-        pos_min="-2.9671" pos_max="2.9671"
-        vel_min="-2.4435" vel_max="2.4435"/>
-      <xacro:joint_ros2_control name="joint4"
-        initial_position="${initial_positions['joint4']}"
-        pos_min="-1.8675" pos_max="2.6878"
-        vel_min="-2.4435" vel_max="2.4435"/>
-      <xacro:joint_ros2_control name="joint5"
-        initial_position="${initial_positions['joint5']}"
-        pos_min="-2.9671" pos_max="2.9671"
-        vel_min="-4.8869" vel_max="4.8869"/>
-      <xacro:joint_ros2_control name="joint6"
-        initial_position="${initial_positions['joint6']}"
-        pos_min="-1.3963" pos_max="4.5379"
-        vel_min="-4.8869" vel_max="4.8869"/>
-      <xacro:joint_ros2_control name="joint7"
-        initial_position="${initial_positions['joint7']}"
-        pos_min="-2.9671" pos_max="2.9671"
-        vel_min="-4.8869" vel_max="4.8869"/>
+      <joint name="${prefix}joint1">
+        <command_interface name="position">
+          <param name="min">-2.7925</param>
+          <param name="max">2.7925</param>
+        </command_interface>
+        <command_interface name="velocity">
+          <param name="min">-2.0944</param>
+          <param name="max">2.0944</param>
+        </command_interface>
+        <command_interface name="effort"/>
+        <state_interface name="position">
+          <!-- initial position for the FakeSystem -->
+          <param name="initial_value">${initial_positions['joint1']}</param>
+        </state_interface>
+        <state_interface name="velocity"/>
+        <state_interface name="effort"/>
+      </joint>
+      <joint name="${prefix}joint2">
+        <command_interface name="position">
+          <param name="min">-2.2689</param>
+          <param name="max">2.2689</param>
+        </command_interface>
+        <command_interface name="velocity">
+          <param name="min">-2.0944</param>
+          <param name="max">2.0944</param>
+        </command_interface>
+        <command_interface name="effort"/>
+        <state_interface name="position">
+          <!-- initial position for the FakeSystem -->
+          <param name="initial_value">${initial_positions['joint2']}</param>
+        </state_interface>
+        <state_interface name="velocity"/>
+        <state_interface name="effort"/>
+      </joint>
+      <joint name="${prefix}joint3">
+        <command_interface name="position">
+          <param name="min">-2.9671</param>
+          <param name="max">2.9671</param>
+        </command_interface>
+        <command_interface name="velocity">
+          <param name="min">-2.4435</param>
+          <param name="max">2.4435</param>
+        </command_interface>
+        <command_interface name="effort"/>
+        <state_interface name="position">
+          <!-- initial position for the FakeSystem -->
+          <param name="initial_value">${initial_positions['joint3']}</param>
+        </state_interface>
+        <state_interface name="velocity"/>
+        <state_interface name="effort"/>
+      </joint>
+      <joint name="${prefix}joint4">
+        <command_interface name="position">
+          <param name="min">-1.8675</param>
+          <param name="max">2.6878</param>
+        </command_interface>
+        <command_interface name="velocity">
+          <param name="min">-2.4435</param>
+          <param name="max">2.4435</param>
+        </command_interface>
+        <command_interface name="effort"/>
+        <state_interface name="position">
+          <!-- initial position for the FakeSystem -->
+          <param name="initial_value">${initial_positions['joint4']}</param>
+        </state_interface>
+        <state_interface name="velocity"/>
+        <state_interface name="effort"/>
+      </joint>
+      <joint name="${prefix}joint5">
+        <command_interface name="position">
+          <param name="min">-2.9671</param>
+          <param name="max">2.9671</param>
+        </command_interface>
+        <command_interface name="velocity">
+          <param name="min">-4.8869</param>
+          <param name="max">4.8869</param>
+        </command_interface>
+        <command_interface name="effort"/>
+        <state_interface name="position">
+          <!-- initial position for the FakeSystem -->
+          <param name="initial_value">${initial_positions['joint5']}</param>
+        </state_interface>
+        <state_interface name="velocity"/>
+        <state_interface name="effort"/>
+      </joint>
+      <joint name="${prefix}joint6">
+        <command_interface name="position">
+          <param name="min">-1.3963</param>
+          <param name="max">4.5379</param>
+        </command_interface>
+        <command_interface name="velocity">
+          <param name="min">-4.8869</param>
+          <param name="max">4.8869</param>
+        </command_interface>
+        <command_interface name="effort"/>
+        <state_interface name="position">
+          <!-- initial position for the FakeSystem -->
+          <param name="initial_value">${initial_positions['joint6']}</param>
+        </state_interface>
+        <state_interface name="velocity"/>
+        <state_interface name="effort"/>
+      </joint>
+      <joint name="${prefix}joint7">
+        <command_interface name="position">
+          <param name="min">-2.9671</param>
+          <param name="max">2.9671</param>
+        </command_interface>
+        <command_interface name="velocity">
+          <param name="min">-4.8869</param>
+          <param name="max">4.8869</param>
+        </command_interface>
+        <command_interface name="effort"/>
+        <state_interface name="position">
+          <!-- initial position for the FakeSystem -->
+          <param name="initial_value">${initial_positions['joint7']}</param>
+        </state_interface>
+        <state_interface name="velocity"/>
+        <state_interface name="effort"/>
+      </joint>
       <!-- 18 digital IO ports (16 on control box + 2 inside the wrist connector) -->
       <gpio name="${prefix}gpio">

File: flexiv_description/urdf/rizon_macro.xacro (robot description, xacro)
@@ -12,4 +12,5 @@
     add_world:=true
     parent:=world
+    mujoco_model
     ">
     <!-- Load gripper -->
@@ -28,10 +29,21 @@
       </xacro:rizon4_joints_links>
       <!-- ros2 control include -->
-      <xacro:include filename="$(find flexiv_description)/urdf/rizon4.ros2_control.xacro"/>
-      <xacro:rizon4_ros2_control prefix="${prefix}" robot_sn="${robot_sn}"
-        use_fake_hardware="${use_fake_hardware}"
-        fake_sensor_commands="${fake_sensor_commands}"
-        initial_positions="${initial_positions}"
-        />
+      <xacro:if value="${mujoco_model==''}">
+        <xacro:include filename="$(find flexiv_description)/urdf/rizon4.ros2_control.xacro"/>
+        <xacro:rizon4_ros2_control prefix="${prefix}" robot_sn="${robot_sn}"
+          use_fake_hardware="${use_fake_hardware}"
+          fake_sensor_commands="${fake_sensor_commands}"
+          initial_positions="${initial_positions}"
+          />
+      </xacro:if>
+      <xacro:unless value="${mujoco_model==''}">
+        <xacro:include filename="$(find flexiv_description)/urdf/rizon_mujoco.ros2_control.xacro"/>
+        <xacro:rizon_mujoco_ros2_control prefix="${prefix}" robot_sn="${robot_sn}"
+          use_fake_hardware="${use_fake_hardware}"
+          fake_sensor_commands="${fake_sensor_commands}"
+          initial_positions="${initial_positions}"
+          mujoco_model="${mujoco_model}"
+          />
+      </xacro:unless>
     </xacro:if>
     <!-- Rizon 10 or 10s-->
